File: KiCAD/PCB/Henge40_PCB.kicad_sch (KiCad schematic)
At the start: 85 parts, among them SW1 SW_Push, SW10 SW_Push, SW11 SW_Push, SW12 SW_Push, SW13 SW_Push, SW14 SW_Push, SW15 SW_Push, SW16 SW_Push, SW17 SW_Push, SW18 SW_Push, SW19 SW_Push, SW2 SW_Push, SW20 SW_Push, SW21 SW_Push, SW21_1 SW_Push, SW22 SW_Push, SW23 SW_Push, SW24 SW_Push, SW25 SW_Push, SW26 SW_Push, SW27 SW_Push, SW28 SW_Push, SW29 SW_Push, SW3 SW_Push, SW30 SW_Push, SW31 SW_Push, SW31_1 SW_Push, SW32 SW_Push, SW33 SW_Push, SW34 SW_Push, SW35 SW_Push, SW36 SW_Push, SW37 SW_Push, SW38 SW_Push, SW39 SW_Push, SW4 SW_Push, SW40 SW_Push, SW41 SW_Push, SW5 SW_Push, SW6 SW_Push, SW7 SW_Push, SW8 SW_Push, SW9 SW_Push, U1 rp2040-tiny

Commit message: 1stロット量産断面
Parts:
- SW1, SW10, SW11, SW12, SW13, SW14, SW15, SW16, SW17, SW18, SW19, SW2, SW20, SW21, SW21_1, SW22, SW23, SW24, SW25, SW26, SW27, SW28, SW29, SW3, SW30, SW31, SW31_1, SW32, SW33, SW34, SW35, SW36, SW37, SW38, SW39, SW4, SW40, SW41, SW5, SW6, SW7, SW8, SW9: LCSC Parts # (none) -> C18212911
Changed lines of the file:
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@@
       (effects (font (size 1.27 1.27)) hide)
     )
-    (property "LCSC Parts #" "" (at 59.69 41.91 0)
+    (property "LCSC Parts #" "C18212911" (at 59.69 41.91 0)
       (effects (font (size 1.27 1.27)) hide)
     )
@@
       (effects (font (size 1.27 1.27)) hide)
     )
-    (property "LCSC Parts #" "" (at 36.83 58.42 0)
+    (property "LCSC Parts #" "C18212911" (at 36.83 58.42 0)
       (effects (font (size 1.27 1.27)) hide)
     )
@@
       (effects (font (size 1.27 1.27)) hide)
     )
-    (property "LCSC Parts #" "" (at 82.55 58.42 0)
+    (property "LCSC Parts #" "C18212911" (at 82.55 58.42 0)
       (effects (font (size 1.27 1.27)) hide)
     )
@@
       (effects (font (size 1.27 1.27)) hide)
     )
-    (property "LCSC Parts #" "" (at 59.69 58.42 0)
+    (property "LCSC Parts #" "C18212911" (at 59.69 58.42 0)
       (effects (font (size 1.27 1.27)) hide)
     )
@@
       (effects (font (size 1.27 1.27)) hide)
     )
-    (property "LCSC Parts #" "" (at 59.69 93.98 0)
+    (property "LCSC Parts #" "C18212911" (at 59.69 93.98 0)
       (effects (font (size 1.27 1.27)) hide)
     )
@@
       (effects (font (size 1.27 1.27)) hide)
     )
-    (property "LCSC Parts #" "" (at 36.83 74.93 0)
+    (property "LCSC Parts #" "C18212911" (at 36.83 74.93 0)
       (effects (font (size 1.27 1.27)) hide)
     )
@@
       (effects (font (size 1.27 1.27)) hide)
     )
-    (property "LCSC Parts #" "" (at 219.71 41.91 0)
+    (property "LCSC Parts #" "C18212911" (at 219.71 41.91 0)
       (effects (font (size 1.27 1.27)) hide)
     )
@@
       (effects (font (size 1.27 1.27)) hide)
     )
-    (property "LCSC Parts #" "" (at 151.13 93.98 0)
+    (property "LCSC Parts #" "C18212911" (at 151.13 93.98 0)
       (effects (font (size 1.27 1.27)) hide)
     )
@@
       (effects (font (size 1.27 1.27)) hide)
     )
-    (property "LCSC Parts #" "" (at 59.69 74.93 0)
+    (property "LCSC Parts #" "C18212911" (at 59.69 74.93 0)
       (effects (font (size 1.27 1.27)) hide)
     )
@@
       (effects (font (size 1.27 1.27)) hide)
     )
-    (property "LCSC Parts #" "" (at 36.83 41.91 0)
+    (property "LCSC Parts #" "C18212911" (at 36.83 41.91 0)
       (effects (font (size 1.27 1.27)) hide)
     )
@@
       (effects (font (size 1.27 1.27)) hide)
     )
-    (property "LCSC Parts #" "" (at 242.57 41.91 0)
+    (property "LCSC Parts #" "C18212911" (at 242.57 41.91 0)
       (effects (font (size 1.27 1.27)) hide)
     )
@@
       (effects (font (size 1.27 1.27)) hide)
     )
-    (property "LCSC Parts #" "" (at 82.55 74.93 0)
+    (property "LCSC Parts #" "C18212911" (at 82.55 74.93 0)
       (effects (font (size 1.27 1.27)) hide)
     )
@@
       (effects (font (size 1.27 1.27)) hide)
     )
-    (property "LCSC Parts #" "" (at 173.99 58.42 0)
+    (property "LCSC Parts #" "C18212911" (at 173.99 58.42 0)
       (effects (font (size 1.27 1.27)) hide)
     )
@@
       (effects (font (size 1.27 1.27)) hide)
     )
-    (property "LCSC Parts #" "" (at 229.87 93.98 0)
+    (property "LCSC Parts #" "C18212911" (at 229.87 93.98 0)
       (effects (font (size 1.27 1.27)) hide)
     )
@@
       (effects (font (size 1.27 1.27)) hide)
     )
-    (property "LCSC Parts #" "" (at 219.71 58.42 0)
+    (property "LCSC Parts #" "C18212911" (at 219.71 58.42 0)
       (effects (font (size 1.27 1.27)) hide)
     )
@@
       (effects (font (size 1.27 1.27)) hide)
     )
-    (property "LCSC Parts #" "" (at 161.29 93.98 0)
+    (property "LCSC Parts #" "C18212911" (at 161.29 93.98 0)
       (effects (font (size 1.27 1.27)) hide)
     )
@@
       (effects (font (size 1.27 1.27)) hide)
     )
-    (property "LCSC Parts #" "" (at 242.57 58.42 0)
+    (property "LCSC Parts #" "C18212911" (at 242.57 58.42 0)
       (effects (font (size 1.27 1.27)) hide)
     )
@@
       (effects (font (size 1.27 1.27)) hide)
     )
-    (property "LCSC Parts #" "" (at 173.99 74.93 0)
+    (property "LCSC Parts #" "C18212911" (at 173.99 74.93 0)
       (effects (font (size 1.27 1.27)) hide)
     )
@@
       (effects (font (size 1.27 1.27)) hide)
     )
-    (property "LCSC Parts #" "" (at 196.85 58.42 0)
+    (property "LCSC Parts #" "C18212911" (at 196.85 58.42 0)
       (effects (font (size 1.27 1.27)) hide)
     )
@@
       (effects (font (size 1.27 1.27)) hide)
     )
-    (property "LCSC Parts #" "" (at 105.41 74.93 0)
+    (property "LCSC Parts #" "C18212911" (at 105.41 74.93 0)
       (effects (font (size 1.27 1.27)) hide)
     )
@@
       (effects (font (size 1.27 1.27)) hide)
     )
-    (property "LCSC Parts #" "" (at 242.57 93.98 0)
+    (property "LCSC Parts #" "C18212911" (at 242.57 93.98 0)
       (effects (font (size 1.27 1.27)) hide)
     )
@@
       (effects (font (size 1.27 1.27)) hide)
     )
-    (property "LCSC Parts #" "" (at 265.43 41.91 0)
+    (property "LCSC Parts #" "C18212911" (at 265.43 41.91 0)
       (effects (font (size 1.27 1.27)) hide)
     )
@@
       (effects (font (size 1.27 1.27)) hide)
     )
-    (property "LCSC Parts #" "" (at 196.85 41.91 0)
+    (property "LCSC Parts #" "C18212911" (at 196.85 41.91 0)
       (effects (font (size 1.27 1.27)) hide)
     )
@@
       (effects (font (size 1.27 1.27)) hide)
     )
-    (property "LCSC Parts #" "" (at 105.41 58.42 0)
+    (property "LCSC Parts #" "C18212911" (at 105.41 58.42 0)
       (effects (font (size 1.27 1.27)) hide)
     )
@@
       (effects (font (size 1.27 1.27)) hide)
     )
-    (property "LCSC Parts #" "" (at 196.85 74.93 0)
+    (property "LCSC Parts #" "C18212911" (at 196.85 74.93 0)
       (effects (font (size 1.27 1.27)) hide)
     )
@@
       (effects (font (size 1.27 1.27)) hide)
     )
-    (property "LCSC Parts #" "" (at 288.29 58.42 0)
+    (property "LCSC Parts #" "C18212911" (at 288.29 58.42 0)
       (effects (font (size 1.27 1.27)) hide)
     )
@@
       (effects (font (size 1.27 1.27)) hide)
     )
-    (property "LCSC Parts #" "" (at 105.41 93.98 0)
+    (property "LCSC Parts #" "C18212911" (at 105.41 93.98 0)
       (effects (font (size 1.27 1.27)) hide)
     )
@@
       (effects (font (size 1.27 1.27)) hide)
     )
-    (property "LCSC Parts #" "" (at 219.71 74.93 0)
+    (property "LCSC Parts #" "C18212911" (at 219.71 74.93 0)
       (effects (font (size 1.27 1.27)) hide)
     )
@@
       (effects (font (size 1.27 1.27)) hide)
     )
-    (property "LCSC Parts #" "" (at 265.43 58.42 0)
+    (property "LCSC Parts #" "C18212911" (at 265.43 58.42 0)
       (effects (font (size 1.27 1.27)) hide)
     )
@@
       (effects (font (size 1.27 1.27)) hide)
     )
-    (property "LCSC Parts #" "" (at 219.71 93.98 0)
+    (property "LCSC Parts #" "C18212911" (at 219.71 93.98 0)
       (effects (font (size 1.27 1.27)) hide)
     )
@@
       (effects (font (size 1.27 1.27)) hide)
     )
-    (property "LCSC Parts #" "" (at 151.13 41.91 0)
+    (property "LCSC Parts #" "C18212911" (at 151.13 41.91 0)
       (effects (font (size 1.27 1.27)) hide)
     )
@@
       (effects (font (size 1.27 1.27)) hide)
     )
-    (property "LCSC Parts #" "" (at 242.57 74.93 0)
+    (property "LCSC Parts #" "C18212911" (at 242.57 74.93 0)
       (effects (font (size 1.27 1.27)) hide)
     )
@@
       (effects (font (size 1.27 1.27)) hide)
     )
-    (property "LCSC Parts #" "" (at 288.29 74.93 0)
+    (property "LCSC Parts #" "C18212911" (at 288.29 74.93 0)
       (effects (font (size 1.27 1.27)) hide)
     )
@@
       (effects (font (size 1.27 1.27)) hide)
     )
-    (property "LCSC Parts #" "" (at 105.41 41.91 0)
+    (property "LCSC Parts #" "C18212911" (at 105.41 41.91 0)
       (effects (font (size 1.27 1.27)) hide)
     )
@@
       (effects (font (size 1.27 1.27)) hide)
     )
-    (property "LCSC Parts #" "" (at 82.55 41.91 0)
+    (property "LCSC Parts #" "C18212911" (at 82.55 41.91 0)
       (effects (font (size 1.27 1.27)) hide)
     )
@@
       (effects (font (size 1.27 1.27)) hide)
     )
-    (property "LCSC Parts #" "" (at 173.99 41.91 0)
+    (property "LCSC Parts #" "C18212911" (at 173.99 41.91 0)
       (effects (font (size 1.27 1.27)) hide)
     )
@@
       (effects (font (size 1.27 1.27)) hide)
     )
-    (property "LCSC Parts #" "" (at 128.27 58.42 0)
+    (property "LCSC Parts #" "C18212911" (at 128.27 58.42 0)
       (effects (font (size 1.27 1.27)) hide)
     )
@@
       (effects (font (size 1.27 1.27)) hide)
     )
-    (property "LCSC Parts #" "" (at 128.27 41.91 0)
+    (property "LCSC Parts #" "C18212911" (at 128.27 41.91 0)
       (effects (font (size 1.27 1.27)) hide)
     )
@@
       (effects (font (size 1.27 1.27)) hide)
     )
-    (property "LCSC Parts #" "" (at 151.13 74.93 0)
+    (property "LCSC Parts #" "C18212911" (at 151.13 74.93 0)
       (effects (font (size 1.27 1.27)) hide)
     )
@@
       (effects (font (size 1.27 1.27)) hide)
     )
-    (property "LCSC Parts #" "" (at 151.13 58.42 0)
+    (property "LCSC Parts #" "C18212911" (at 151.13 58.42 0)
       (effects (font (size 1.27 1.27)) hide)
     )
@@
       (effects (font (size 1.27 1.27)) hide)
     )
-    (property "LCSC Parts #" "" (at 288.29 41.91 0)
+    (property "LCSC Parts #" "C18212911" (at 288.29 41.91 0)
       (effects (font (size 1.27 1.27)) hide)
     )
@@
       (effects (font (size 1.27 1.27)) hide)
     )
-    (property "LCSC Parts #" "" (at 128.27 74.93 0)
+    (property "LCSC Parts #" "C18212911" (at 128.27 74.93 0)
       (effects (font (size 1.27 1.27)) hide)
     )
@@
       (effects (font (size 1.27 1.27)) hide)
     )
-    (property "LCSC Parts #" "" (at 265.43 74.93 0)
-      (effects (font (size 1.27 1.27)) hide)
-    )
+    (property "LCSC Parts #" "C18212911" (at 265.43 74.93 0)
+      (effects (font (size 1.27 1.27)) hide)
+    )
